Commit message: added the ros2_control to robotic arm

File: robotic_arm_description/urdf/robotic_arm.xacro (robot description, xacro)
@@ -2,4 +2,6 @@
 <robot name="robotic_arm" xmlns:xacro="http://www.ros.org/wiki/xacro">
   <xacro:include filename="materials.xacro"/>
+  <xacro:include filename="$(find robotic_arm_description)/urdf/robotic_arm_gazebo.xacro"/>
+  <xacro:include filename="$(find robotic_arm_description)/urdf/robotic_arm_ros2_control.xacro"/>
   <!-- Useful XACRO Variables (Properties) -->
   <xacro:property name="PI" value="3.14159265359" />
@@ -688,3 +690,38 @@
     <child link="right_arm_1" />
   </joint>
+  <transmission name="transmission_base">
+    <plugin>transmission_interface/SimpleTransmission</plugin>
+    <actuator name="base_servo" role="actuator1"/>
+    <joint name="Base Rotate" role="joint1">
+        <mechanical_reduction>1.0</mechanical_reduction>
+    </joint>
+  </transmission>
+  <transmission name="transmission_shoulder">
+    <plugin>transmission_interface/SimpleTransmission</plugin>
+    <actuator name="shoulder_servo" role="actuator1"/>
+    <joint name="Shoulder Rotate" role="joint1">
+        <mechanical_reduction>1.0</mechanical_reduction>
+    </joint>
+  </transmission>
+  <transmission name="transmission_elbow">
+    <plugin>transmission_interface/SimpleTransmission</plugin>
+    <actuator name="elbow_servo" role="actuator1"/>
+    <joint name="Elbow Rotate" role="joint1">
+        <mechanical_reduction>1.0</mechanical_reduction>
+    </joint>
+  </transmission>
+  <transmission name="transmission_wrist">
+    <plugin>transmission_interface/SimpleTransmission</plugin>
+    <actuator name="wrist_servo" role="actuator1"/>
+    <joint name="Wrist Rotate" role="joint1">
+        <mechanical_reduction>1.0</mechanical_reduction>
+    </joint>
+  </transmission>
+  <transmission name="transmission_grab">
+    <plugin>transmission_interface/SimpleTransmission</plugin>
+    <actuator name="grab_servo" role="actuator1"/>
+    <joint name="Gripper Grab" role="joint1">
+        <mechanical_reduction>1.0</mechanical_reduction>
+    </joint>
+  </transmission>
 </robot>
