Commit message: ros2_control to main robot

File: ros_robot_description/urdf/ros_robot.xacro (robot description, xacro)
@@ -2,4 +2,6 @@
 <robot name="ros_robot" xmlns:xacro="http://www.ros.org/wiki/xacro">
   <xacro:include filename="materials.xacro"/>
+  <xacro:include filename="$(find ros_robot_description)/urdf/ros_robot_gazebo.xacro"/>
+  <xacro:include filename="$(find ros_robot_description)/urdf/ros_robot_ros2_control.xacro"/>
   <!-- Useful XACRO Variables (Properties) -->
   <xacro:property name="PI" value="3.14159265359" />
@@ -1120,3 +1122,38 @@
     <mimic joint="Gripper Grab" multiplier="-1"/>
   </joint>
+  <transmission name="transmission_base">
+    <plugin>transmission_interface/SimpleTransmission</plugin>
+    <actuator name="base_servo" role="actuator1"/>
+    <joint name="Base Rotate" role="joint1">
+        <mechanical_reduction>1.0</mechanical_reduction>
+    </joint>
+  </transmission>
+  <transmission name="transmission_shoulder">
+    <plugin>transmission_interface/SimpleTransmission</plugin>
+    <actuator name="shoulder_servo" role="actuator1"/>
+    <joint name="Shoulder Rotate" role="joint1">
+        <mechanical_reduction>1.0</mechanical_reduction>
+    </joint>
+  </transmission>
+  <transmission name="transmission_elbow">
+    <plugin>transmission_interface/SimpleTransmission</plugin>
+    <actuator name="elbow_servo" role="actuator1"/>
+    <joint name="Elbow Rotate" role="joint1">
+        <mechanical_reduction>1.0</mechanical_reduction>
+    </joint>
+  </transmission>
+  <transmission name="transmission_wrist">
+    <plugin>transmission_interface/SimpleTransmission</plugin>
+    <actuator name="wrist_servo" role="actuator1"/>
+    <joint name="Wrist Rotate" role="joint1">
+        <mechanical_reduction>1.0</mechanical_reduction>
+    </joint>
+  </transmission>
+  <transmission name="transmission_grab">
+    <plugin>transmission_interface/SimpleTransmission</plugin>
+    <actuator name="grab_servo" role="actuator1"/>
+    <joint name="Gripper Grab" role="joint1">
+        <mechanical_reduction>1.0</mechanical_reduction>
+    </joint>
+  </transmission>
 </robot>

Commit message: teleop_added

File: ros_robot_description/urdf/ros_robot.xacro (robot description, xacro)
@@ -1,7 +1,7 @@
 <?xml version="1.0"?>
 <robot name="ros_robot" xmlns:xacro="http://www.ros.org/wiki/xacro">
-  <xacro:include filename="materials.xacro"/>
-  <xacro:include filename="$(find ros_robot_description)/urdf/ros_robot_gazebo.xacro"/>
-  <xacro:include filename="$(find ros_robot_description)/urdf/ros_robot_ros2_control.xacro"/>
+  <xacro:include filename="materials.xacro" />
+  <xacro:include filename="$(find ros_robot_description)/urdf/ros_robot_gazebo.xacro" />
+  <xacro:include filename="$(find ros_robot_description)/urdf/ros_robot_ros2_control.xacro" />
   <!-- Useful XACRO Variables (Properties) -->
   <xacro:property name="PI" value="3.14159265359" />
@@ -801,4 +801,5 @@
     </collision>
   </link>
+  <link name="camera_link_optical"></link>
   <link name="end_effector_right_1">
     <inertial>
@@ -1088,8 +1089,13 @@
     <child link="gripper_servo_1" />
   </joint>
-  <joint name="Rigid 36" type="fixed">
+  <joint name="camera_joint" type="fixed">
     <origin xyz="0.027475 -0.025918 0.245726" rpy="0 0 0" />
     <parent link="wrist_end_plate_1" />
     <child link="camera_1" />
+  </joint>
+  <joint name="camera_optical_joint" type="fixed">
+    <origin xyz="0 0 0" rpy="${-pi/2} 0 ${-pi/2}" />
+    <parent link="camera_1" />
+    <child link="camera_link_optical" />
   </joint>
   <joint name="Rigid 39" type="fixed">
@@ -1120,69 +1126,101 @@
     <child link="right_gripper_gear_1" />
     <axis xyz="-0.087156 0.0 0.996195" />
-    <mimic joint="Gripper Grab" multiplier="-1"/>
+    <mimic joint="Gripper Grab" multiplier="-1" />
   </joint>
   <transmission name="transmission_base">
     <plugin>transmission_interface/SimpleTransmission</plugin>
-    <actuator name="base_servo" role="actuator1"/>
+    <actuator name="base_servo" role="actuator1" />
     <joint name="Base Rotate" role="joint1">
-        <mechanical_reduction>1.0</mechanical_reduction>
+      <mechanical_reduction>1.0</mechanical_reduction>
     </joint>
   </transmission>
   <transmission name="transmission_shoulder">
     <plugin>transmission_interface/SimpleTransmission</plugin>
-    <actuator name="shoulder_servo" role="actuator1"/>
+    <actuator name="shoulder_servo" role="actuator1" />
     <joint name="Shoulder Rotate" role="joint1">
-        <mechanical_reduction>1.0</mechanical_reduction>
+      <mechanical_reduction>1.0</mechanical_reduction>
     </joint>
   </transmission>
   <transmission name="transmission_elbow">
     <plugin>transmission_interface/SimpleTransmission</plugin>
-    <actuator name="elbow_servo" role="actuator1"/>
+    <actuator name="elbow_servo" role="actuator1" />
     <joint name="Elbow Rotate" role="joint1">
-        <mechanical_reduction>1.0</mechanical_reduction>
+      <mechanical_reduction>1.0</mechanical_reduction>
     </joint>
   </transmission>
   <transmission name="transmission_wrist">
     <plugin>transmission_interface/SimpleTransmission</plugin>
-    <actuator name="wrist_servo" role="actuator1"/>
+    <actuator name="wrist_servo" role="actuator1" />
     <joint name="Wrist Rotate" role="joint1">
-        <mechanical_reduction>1.0</mechanical_reduction>
+      <mechanical_reduction>1.0</mechanical_reduction>
     </joint>
   </transmission>
   <transmission name="transmission_grab">
     <plugin>transmission_interface/SimpleTransmission</plugin>
-    <actuator name="grab_servo" role="actuator1"/>
+    <actuator name="grab_servo" role="actuator1" />
     <joint name="Gripper Grab" role="joint1">
-        <mechanical_reduction>1.0</mechanical_reduction>
+      <mechanical_reduction>1.0</mechanical_reduction>
     </joint>
   </transmission>
   <gazebo reference="lidar_scan_1">
-      <sensor name="laser" type="ray">
-          <pose>0 0 0 0 0 0</pose>
-          <visualize>true</visualize>
-          <update_rate>10</update_rate>
-          <ray>
-              <scan>
-                  <horizontal>
-                      <samples>360</samples>
-                      <resolution>1</resolution>
-                      <min_angle>-3.14</min_angle>
-                      <max_angle>3.14</max_angle>
-                  </horizontal>
-              </scan>
-              <range>
-                  <min>0.3</min>
-                  <max>12</max>
-                  <resolution>0.01</resolution>
-              </range>
-          </ray>
-          <plugin name="laser_controller" filename="libgazebo_ros_ray_sensor.so">
-              <ros>
-                  <argument>~/out:=scan</argument>
-              </ros>
-              <output_type>sensor_msgs/LaserScan</output_type>
-              <frame_name>lidar_scan_1</frame_name>
-          </plugin>
-      </sensor>
+    <sensor name="laser" type="ray">
+      <pose>0 0 0 0 0 0</pose>
+      <visualize>true</visualize>
+      <update_rate>10</update_rate>
+      <ray>
+        <scan>
+          <horizontal>
+            <samples>360</samples>
+            <resolution>1</resolution>
+            <min_angle>-3.14</min_angle>
+            <max_angle>3.14</max_angle>
+          </horizontal>
+        </scan>
+        <range>
+          <min>0.3</min>
+          <max>12</max>
+          <resolution>0.01</resolution>
+        </range>
+      </ray>
+      <plugin name="laser_controller" filename="libgazebo_ros_ray_sensor.so">
+        <ros>
+          <argument>~/out:=scan</argument>
+        </ros>
+        <output_type>sensor_msgs/LaserScan</output_type>
+        <frame_name>lidar_scan_1</frame_name>
+      </plugin>
+    </sensor>
+  </gazebo>
+  <gazebo reference="camera_1">
+    <sensor name="camera" type="camera">
+      <pose>0 0 0 0 0 0</pose>
+      <visualize>true</visualize>
+      <update_rate>10</update_rate>
+      <camera>
+        <horizontal_fov>1.089</horizontal_fov>
+        <image>
+          <format>R8G8B8</format>
+          <width>640</width>
+          <height>480</height>
+        </image>
+        <clip>
+          <near>0.05</near>
+          <far>8.0</far>
+        </clip>
+      </camera>
+      <plugin name="camera_controller" filename="libgazebo_ros_camera.so">
+        <frame_name>camera_link_optical</frame_name>
+      </plugin>
+    </sensor>
+  </gazebo>
+  <gazebo>
+    <plugin name="my_mecanum_drive_controller" filename="libgazebo_ros_planar_move.so">
+      <commandTopic>cmd_vel</commandTopic>
+      <odometryTopic>odom</odometryTopic>
+      <odometryFrame>odom</odometryFrame>
+      <odometryRate>50.0</odometryRate>
+      <robotBaseFrame>base_link</robotBaseFrame>
+      <publishTF>false</publishTF>
+    </plugin>
   </gazebo>
 </robot>

Commit message: gazebo colors fixed

File: ros_robot_description/urdf/ros_robot.xacro (robot description, xacro)
@@ -1224,3 +1224,126 @@
     </plugin>
   </gazebo>
+  <gazebo reference="base_link">
+    <material>Gazebo/Green</material>
+  </gazebo>
+  <gazebo reference="motor_1_1">
+    <material>Gazebo/Gray</material>
+  </gazebo>
+  <gazebo reference="motor_2_1">
+    <material>Gazebo/Gray</material>
+  </gazebo>
+  <gazebo reference="motor_3_1">
+    <material>Gazebo/Gray</material>
+  </gazebo>
+  <gazebo reference="motor_4_1">
+    <material>Gazebo/Gray</material>
+  </gazebo>
+  <gazebo reference="coupling_1_1">
+    <material>Gazebo/Yellow</material>
+  </gazebo>
+  <gazebo reference="coupling_2_1">
+    <material>Gazebo/Yellow</material>
+  </gazebo>
+  <gazebo reference="coupling_3_1">
+    <material>Gazebo/Yellow</material>
+  </gazebo>
+  <gazebo reference="coupling_4_1">
+    <material>Gazebo/Yellow</material>
+  </gazebo>
+  <gazebo reference="wheel_1_1">
+    <material>Gazebo/Black</material>
+  </gazebo>
+  <gazebo reference="wheel_2_1">
+    <material>Gazebo/Black</material>
+  </gazebo>
+  <gazebo reference="wheel_3_1">
+    <material>Gazebo/Black</material>
+  </gazebo>
+  <gazebo reference="wheel_4_1">
+    <material>Gazebo/Black</material>
+  </gazebo>
+  <gazebo reference="lidar_base_1">
+    <material>Gazebo/Black</material>
+  </gazebo>
+  <gazebo reference="lidar_scan_1">
+    <material>Gazebo/Blue</material>
+  </gazebo>
+  <gazebo reference="tf_luna_1">
+    <material>Gazebo/Black</material>
+  </gazebo>
+  <gazebo reference="servo_base_plate_1">
+    <material>Gazebo/Yellow</material>
+  </gazebo>
+  <gazebo reference="base_servo_1">
+    <material>Gazebo/Black</material>
+  </gazebo>
+  <gazebo reference="base_horn_1">
+    <material>Gazebo/Gray</material>
+  </gazebo>
+  <gazebo reference="base_servo_rotate_plate_1">
+    <material>Gazebo/Yellow</material>
+  </gazebo>
+  <gazebo reference="servo_1_horn_1_1">
+    <material>Gazebo/Gray</material>
+  </gazebo>
+  <gazebo reference="servo_1_horn_2_1">
+    <material>Gazebo/Gray</material>
+  </gazebo>
+  <gazebo reference="middle_plate_lower_1">
+    <material>Gazebo/Yellow</material>
+  </gazebo>
+  <gazebo reference="middle_plate_upper_1">
+    <material>Gazebo/Yellow</material>
+  </gazebo>
+  <gazebo reference="servo_2_horn_1_1">
+    <material>Gazebo/Gray</material>
+  </gazebo>
+  <gazebo reference="servo_2_horn_2_1">
+    <material>Gazebo/Gray</material>
+  </gazebo>
+  <gazebo reference="servo_2_1">
+    <material>Gazebo/Black</material>
+  </gazebo>
+  <gazebo reference="upper_arm_1">
+    <material>Gazebo/Yellow</material>
+  </gazebo>
+  <gazebo reference="wrist_servo_plate_1">
+    <material>Gazebo/Yellow</material>
+  </gazebo>
+  <gazebo reference="servo_3_horn_1_1">
+    <material>Gazebo/Gray</material>
+  </gazebo>
+  <gazebo reference="servo_3_horn_2_1">
+    <material>Gazebo/Gray</material>
+  </gazebo>
+  <gazebo reference="servo_3_1">
+    <material>Gazebo/Black</material>
+  </gazebo>
+  <gazebo reference="wrist_end_plate_1">
+    <material>Gazebo/Yellow</material>
+  </gazebo>
+  <gazebo reference="gripper_plate_1">
+    <material>Gazebo/Yellow</material>
+  </gazebo>
+  <gazebo reference="gripper_servo_1">
+    <material>Gazebo/Black</material>
+  </gazebo>
+  <gazebo reference="camera_1">
+    <material>Gazebo/Blue</material>
+  </gazebo>
+  <gazebo reference="end_effector_right_1">
+    <material>Gazebo/Red</material>
+  </gazebo>
+  <gazebo reference="end_effector_left_1">
+    <material>Gazebo/Red</material>
+  </gazebo>
+  <gazebo reference="servo_1_1">
+    <material>Gazebo/Black</material>
+  </gazebo>
+  <gazebo reference="left_gripper_gear_1">
+    <material>Gazebo/Red</material>
+  </gazebo>
+  <gazebo reference="right_gripper_gear_1">
+    <material>Gazebo/Red</material>
+  </gazebo>
 </robot>

Commit message: odom fixed

File: ros_robot_description/urdf/ros_robot.xacro (robot description, xacro)
@@ -31,4 +31,11 @@
     </collision>
   </link>
+  <link name="base_footprint">
+  </link>
+  <joint name="base_footprint_joint" type="fixed">
+    <parent link="base_footprint"/>
+    <child link="base_link"/>
+    <origin xyz="0 0 0" rpy="0 0 0"/>
+  </joint>
   <link name="motor_1_1">
     <inertial>
@@ -1219,7 +1226,7 @@
       <odometryTopic>odom</odometryTopic>
       <odometryFrame>odom</odometryFrame>
-      <odometryRate>50.0</odometryRate>
-      <robotBaseFrame>base_link</robotBaseFrame>
-      <publishTF>false</publishTF>
+      <odometryRate>20.0</odometryRate>
+      <robotBaseFrame>base_footprint</robotBaseFrame>
+      <publishTF>true</publishTF>
     </plugin>
   </gazebo>

Commit message: sim time

File: ros_robot_description/urdf/ros_robot.xacro (robot description, xacro)
@@ -8,4 +8,13 @@
   <xacro:property name="effort" value="30.0" />
   <xacro:property name="velocity" value="10.0" />
+  <link name ="base_footprint">
+  </link>
+  <joint name="footprint_joint" type="fixed">
+       <origin
+              xyz="0.0 0.0 0.0"
+              rpy="0 0 0" />
+      <parent link="base_footprint"/>
+      <child link="base_link"/>
+  </joint>
   <link name="base_link">
     <inertial>
@@ -31,11 +40,4 @@
     </collision>
   </link>
-  <link name="base_footprint">
-  </link>
-  <joint name="base_footprint_joint" type="fixed">
-    <parent link="base_footprint"/>
-    <child link="base_link"/>
-    <origin xyz="0 0 0" rpy="0 0 0"/>
-  </joint>
   <link name="motor_1_1">
     <inertial>
@@ -1222,11 +1224,10 @@
   </gazebo>
   <gazebo>
-    <plugin name="my_mecanum_drive_controller" filename="libgazebo_ros_planar_move.so">
+    <plugin name="object_controller" filename="libgazebo_ros_planar_move.so">
       <commandTopic>cmd_vel</commandTopic>
       <odometryTopic>odom</odometryTopic>
       <odometryFrame>odom</odometryFrame>
       <odometryRate>20.0</odometryRate>
-      <robotBaseFrame>base_footprint</robotBaseFrame>
-      <publishTF>true</publishTF>
+      <robotBaseFrame>chasis</robotBaseFrame>
     </plugin>
   </gazebo>
